Commit message: feat(pursuit-guidance): add pursuit-evasion guidance environment
- New PursuitGuidanceTask with room walls, static obstacles, and target quadrotor
- ThrustBodyRateController applying direct force/torque commands
- PursuitQuadDirect robot bypassing allocation for root-link control
- PPO training script (ppo_guidance.py) for reinforcement learning
- Updated registries, asset loader, motor model, and control allocation
- use pursuit_quad_direct 99.9% success rate, migration success

File: resources/robots/quad/model.urdf (robot description, URDF)
Before this commit: robot quadrotor, 5 links, 4 joints
Links:
- link base_link: mass 1.2 -> 1.9; geometry collision sphere radius=0.2; visual cylinder length=0.025 radius=0.2
